File: kicad/caret_pcb/caret_piezo_sensor.kicad_sch (KiCad schematic)
At the start: 25 parts, among them Q1 BSS138BK, Q2 BSS138BK, U2 LM324

Commit message: kicad.caret_pcb: add 3d printer boards
Parts:
- C1, C2, C3: value (none) -> 0.1uF; footprint (none) -> Capacitor_SMD:C_0603_1608Metric
- C4, C5: value (none) -> 1 uF 10 V 10%; footprint (none) -> Capacitor_SMD:C_0603_1608Metric
- D3: value (none) -> RED; footprint (none) -> Diode_SMD:D_0805_2012Metric
- D5: value (none) -> BLUE; footprint (none) -> Diode_SMD:D_0805_2012Metric
- R1: value (none) -> 10k; footprint (none) -> Resistor_SMD:R_0603_1608Metric
- R10, R2, R3, R4, R5, R6, R7, R8, R9: footprint (none) -> Resistor_SMD:R_0603_1608Metric
Changed lines of the file:
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@@
       (effects (font (size 1.27 1.27)) (justify right))
     )
-    (property "Value" "" (id 1) (at 185.42 99.4408 90)
-      (effects (font (size 1.27 1.27)) (justify right))
-    )
-    (property "Footprint" "" (id 2) (at 181.61 97.79 0)
+    (property "Value" "RED" (id 1) (at 185.42 99.4408 90)
+      (effects (font (size 1.27 1.27)) (justify right))
+    )
+    (property "Footprint" "Diode_SMD:D_0805_2012Metric" (id 2) (at 181.61 97.79 0)
       (effects (font (size 1.27 1.27)) hide)
     )
@@
       (effects (font (size 1.27 1.27)) (justify right))
     )
-    (property "Value" "" (id 1) (at 165.1 44.4499 0)
-      (effects (font (size 1.27 1.27)) (justify right))
-    )
-    (property "Footprint" "" (id 2) (at 160.3248 39.37 0)
+    (property "Value" "0.1uF" (id 1) (at 165.1 44.4499 0)
+      (effects (font (size 1.27 1.27)) (justify right))
+    )
+    (property "Footprint" "Capacitor_SMD:C_0603_1608Metric" (id 2) (at 160.3248 39.37 0)
       (effects (font (size 1.27 1.27)) hide)
     )
@@
     (in_bom yes) (on_board yes) (fields_autoplaced)
     (property "Reference" "C1" (id 0) (at 109.22 69.85 90))
-    (property "Value" "" (id 1) (at 109.22 72.39 90))
-    (property "Footprint" "" (id 2) (at 113.03 76.5048 0)
+    (property "Value" "0.1uF" (id 1) (at 109.22 72.39 90))
+    (property "Footprint" "Capacitor_SMD:C_0603_1608Metric" (id 2) (at 113.03 76.5048 0)
       (effects (font (size 1.27 1.27)) hide)
     )
@@
     (in_bom yes) (on_board yes) (fields_autoplaced)
     (property "Reference" "C3" (id 0) (at 162.56 74.93 90))
-    (property "Value" "" (id 1) (at 162.56 77.47 90))
-    (property "Footprint" "" (id 2) (at 166.37 81.5848 0)
+    (property "Value" "0.1uF" (id 1) (at 162.56 77.47 90))
+    (property "Footprint" "Capacitor_SMD:C_0603_1608Metric" (id 2) (at 166.37 81.5848 0)
       (effects (font (size 1.27 1.27)) hide)
     )
@@
       (effects (font (size 1.27 1.27)) (justify right))
     )
-    (property "Value" "" (id 1) (at 118.11 146.0499 0)
-      (effects (font (size 1.27 1.27)) (justify right))
-    )
-    (property "Footprint" "" (id 2) (at 113.3348 140.97 0)
+    (property "Value" "1 uF 10 V 10%" (id 1) (at 118.11 146.0499 0)
+      (effects (font (size 1.27 1.27)) (justify right))
+    )
+    (property "Footprint" "Capacitor_SMD:C_0603_1608Metric" (id 2) (at 113.3348 140.97 0)
       (effects (font (size 1.27 1.27)) hide)
     )
@@
     (property "Reference" "R2" (id 0) (at 132.08 62.23 90))
     (property "Value" "330k" (id 1) (at 134.62 62.23 90))
-    (property "Footprint" "" (id 2) (at 140.208 62.23 90)
+    (property "Footprint" "Resistor_SMD:R_0603_1608Metric" (id 2) (at 140.208 62.23 90)
       (effects (font (size 1.27 1.27)) hide)
     )
@@
     (in_bom yes) (on_board yes) (fields_autoplaced)
     (property "Reference" "R1" (id 0) (at 52.07 104.14 90))
-    (property "Value" "" (id 1) (at 52.07 106.68 90))
-    (property "Footprint" "" (id 2) (at 52.07 112.268 90)
+    (property "Value" "10k" (id 1) (at 52.07 106.68 90))
+    (property "Footprint" "Resistor_SMD:R_0603_1608Metric" (id 2) (at 52.07 112.268 90)
       (effects (font (size 1.27 1.27)) hide)
     )
@@
     (property "Reference" "R10" (id 0) (at 254 86.36 90))
     (property "Value" "1k" (id 1) (at 251.46 86.36 90))
-    (property "Footprint" "" (id 2) (at 245.872 86.36 90)
+    (property "Footprint" "Resistor_SMD:R_0603_1608Metric" (id 2) (at 245.872 86.36 90)
       (effects (font (size 1.27 1.27)) hide)
     )
@@
       (effects (font (size 1.27 1.27)) (justify right))
     )
-    (property "Value" "" (id 1) (at 271.78 103.2508 90)
-      (effects (font (size 1.27 1.27)) (justify right))
-    )
-    (property "Footprint" "" (id 2) (at 267.97 101.6 0)
+    (property "Value" "BLUE" (id 1) (at 271.78 103.2508 90)
+      (effects (font (size 1.27 1.27)) (justify right))
+    )
+    (property "Footprint" "Diode_SMD:D_0805_2012Metric" (id 2) (at 267.97 101.6 0)
       (effects (font (size 1.27 1.27)) hide)
     )
@@
     (property "Reference" "R9" (id 0) (at 205.74 95.25 90))
     (property "Value" "1M" (id 1) (at 203.2 95.25 90))
-    (property "Footprint" "" (id 2) (at 197.612 95.25 90)
+    (property "Footprint" "Resistor_SMD:R_0603_1608Metric" (id 2) (at 197.612 95.25 90)
       (effects (font (size 1.27 1.27)) hide)
     )
@@
       (effects (font (size 1.27 1.27)) (justify left))
     )
-    (property "Footprint" "" (id 2) (at 90.932 68.58 90)
+    (property "Footprint" "Resistor_SMD:R_0603_1608Metric" (id 2) (at 90.932 68.58 90)
       (effects (font (size 1.27 1.27)) hide)
     )
@@
       (effects (font (size 1.27 1.27)) (justify right))
     )
-    (property "Value" "" (id 1) (at 203.2 118.1099 0)
-      (effects (font (size 1.27 1.27)) (justify right))
-    )
-    (property "Footprint" "" (id 2) (at 198.4248 113.03 0)
+    (property "Value" "1 uF 10 V 10%" (id 1) (at 203.2 118.1099 0)
+      (effects (font (size 1.27 1.27)) (justify right))
+    )
+    (property "Footprint" "Capacitor_SMD:C_0603_1608Metric" (id 2) (at 198.4248 113.03 0)
       (effects (font (size 1.27 1.27)) hide)
     )
@@
     (property "Reference" "R5" (id 0) (at 109.22 85.09 90))
     (property "Value" "82k" (id 1) (at 109.22 87.63 90))
-    (property "Footprint" "" (id 2) (at 109.22 93.218 90)
+    (property "Footprint" "Resistor_SMD:R_0603_1608Metric" (id 2) (at 109.22 93.218 90)
       (effects (font (size 1.27 1.27)) hide)
     )
@@
     (property "Reference" "R8" (id 0) (at 187.96 82.55 90))
     (property "Value" "510" (id 1) (at 185.42 82.55 90))
-    (property "Footprint" "" (id 2) (at 179.832 82.55 90)
+    (property "Footprint" "Resistor_SMD:R_0603_1608Metric" (id 2) (at 179.832 82.55 90)
       (effects (font (size 1.27 1.27)) hide)
     )
@@
     (property "Reference" "R7" (id 0) (at 151.13 43.18 90))
     (property "Value" "10k" (id 1) (at 148.59 43.18 90))
-    (property "Footprint" "" (id 2) (at 143.002 43.18 90)
+    (property "Footprint" "Resistor_SMD:R_0603_1608Metric" (id 2) (at 143.002 43.18 90)
       (effects (font (size 1.27 1.27)) hide)
     )
@@
     (property "Reference" "R3" (id 0) (at 144.78 80.01 90))
     (property "Value" "390k" (id 1) (at 142.24 80.01 90))
-    (property "Footprint" "" (id 2) (at 136.652 80.01 90)
+    (property "Footprint" "Resistor_SMD:R_0603_1608Metric" (id 2) (at 136.652 80.01 90)
       (effects (font (size 1.27 1.27)) hide)
     )
@@
     (property "Reference" "R6" (id 0) (at 151.13 27.94 90))
     (property "Value" "10k" (id 1) (at 148.59 27.94 90))
-    (property "Footprint" "" (id 2) (at 143.002 27.94 90)
-      (effects (font (size 1.27 1.27)) hide)
-    )
+    (property "Footprint" "Resistor_SMD:R_0603_1608Metric" (id 2) (at 143.002 27.94 90)
+      (effects (font (size 1.27 1.27)) hide)
+    )

Commit message: caret_pcb: fix power line
Parts:
- added U?: (no value), symbol Amplifier_Operational:LM324
Connections:
- net +5V: now also U?.4 (V+)
- net GND: now also U?.11 (V-)
Changed lines of the file:
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@@
+    (effects (font (size 1.27 1.27)) (justify right))
+  )
+  (hierarchical_label "GND" (shape input) (at 245.11 48.26 270)
     (effects (font (size 1.27 1.27)) (justify right))
   )
@@
   )
   (hierarchical_label "+5V" (shape input) (at 114.3 140.97 90)
+    (effects (font (size 1.27 1.27)) (justify left))
+  )
+  (hierarchical_label "+5V" (shape input) (at 245.11 33.02 90)
     (effects (font (size 1.27 1.27)) (justify left))
   )
@@
     (pin "2")
   )
+  (symbol (lib_id "Amplifier_Operational:LM324") (at 247.65 40.64 0) (unit 5)
+    (in_bom yes) (on_board yes) (fields_autoplaced)
+    (property "Reference" "U?" (id 0) (at 246.38 39.3699 0)
+      (effects (font (size 1.27 1.27)) (justify left))
+    )
+    (property "Value" "" (id 1) (at 246.38 41.9099 0)
+      (effects (font (size 1.27 1.27)) (justify left))
+    )
+    (property "Footprint" "" (id 2) (at 246.38 38.1 0)
+      (effects (font (size 1.27 1.27)) hide)
+    )
+    (property "Datasheet" "http://www.ti.com/lit/ds/symlink/lm2902-n.pdf" (id 3) (at 248.92 35.56 0)
+      (effects (font (size 1.27 1.27)) hide)
+    )
+    (pin "1")
+    (pin "2")
+    (pin "3")
+    (pin "5")
+    (pin "6")
+    (pin "7")
+    (pin "10")
+    (pin "8")
+    (pin "9")
+    (pin "12")
+    (pin "13")
+    (pin "14")
+    (pin "11")
+    (pin "4")
+  )
   (symbol (lib_id "Amplifier_Operational:LM324") (at 161.29 105.41 0) (mirror x) (unit 3)

Commit message: caret_pcb: fix piezo sensor power line, fix rpi shield schematic
Parts:
- U1: renamed from U?; value (none) -> LM324
Changed lines of the file:
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@@
   (symbol (lib_id "Amplifier_Operational:LM324") (at 247.65 40.64 0) (unit 5)
     (in_bom yes) (on_board yes) (fields_autoplaced)
-    (property "Reference" "U?" (id 0) (at 246.38 39.3699 0)
+    (property "Reference" "U1" (id 0) (at 246.38 39.3699 0)
       (effects (font (size 1.27 1.27)) (justify left))
     )
-    (property "Value" "" (id 1) (at 246.38 41.9099 0)
+    (property "Value" "LM324" (id 1) (at 246.38 41.9099 0)
       (effects (font (size 1.27 1.27)) (justify left))
     )
