File: kicad/rpi_motor_pcb/mosfet_gpio.kicad_sch (KiCad schematic)
At the start: 6 parts, among them J18 ${SHEETNAME}, Q4 HY1403D

Commit message: rpi_motor_pcb: 6-axis fix diag pin, add en pin
Parts:
- R5: value (none) -> 10k
- R7: value (none) -> 10k; footprint (none) -> Resistor_SMD:R_0805_2012Metric
- U3: value (none) -> 74LVC1G17; footprint (none) -> Package_TO_SOT_SMD:SOT-23-5
Changed lines of the file:
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@@
       (effects (font (size 1.27 1.27)) (justify right))
     )
-    (property "Value" "" (id 1) (at 29.21 44.7039 0)
+    (property "Value" "10k" (id 1) (at 29.21 44.7039 0)
       (effects (font (size 1.27 1.27)) (justify right))
     )
@@
     (in_bom yes) (on_board yes)
     (property "Reference" "U3" (id 0) (at 38.481 31.75 0))
-    (property "Value" "" (id 1) (at 38.354 33.528 0))
-    (property "Footprint" "" (id 2) (at 39.116 39.624 0)
+    (property "Value" "74LVC1G17" (id 1) (at 38.354 33.528 0))
+    (property "Footprint" "Package_TO_SOT_SMD:SOT-23-5" (id 2) (at 39.116 39.624 0)
       (effects (font (size 1.27 1.27)) hide)
     )
@@
     (in_bom yes) (on_board yes) (fields_autoplaced)
     (property "Reference" "R7" (id 0) (at 49.276 33.02 90))
-    (property "Value" "" (id 1) (at 49.276 35.56 90))
-    (property "Footprint" "" (id 2) (at 49.276 41.402 90)
+    (property "Value" "10k" (id 1) (at 49.276 35.56 90))
+    (property "Footprint" "Resistor_SMD:R_0805_2012Metric" (id 2) (at 49.276 41.402 90)
       (effects (font (size 1.27 1.27)) hide)
     )
